File: PCB/DAC ADC PWM IO.kicad_pcb (KiCad board)
At the start: 4 copper layers, 100 x 100 mm, 270 parts, among them J1 Screw_Terminal_01x9, J14 Screw_Terminal_01x15, J15 Screw_Terminal_01x10, J16 Screw_Terminal_01x9, J2 Screw_Terminal_01x02, J3 Conn_01x08, J8 Screw_Terminal_01x12, J9 USB_B, Q1 BC847C-QR, Q10 BUK9M15-60EX, Q11 BUK9M15-60EX, Q2 BC847C-QR, Q3 BC847C-QR, Q4 BUK9M15-60EX, Q5 BUK9M15-60EX, Q6 BUK9M15-60EX, Q7 BUK9M15-60EX, Q8 BUK9M15-60EX, Q9 BUK9M15-60EX, SW1 SW_Push, U2 AP7343-33W5-7, U3 LM2902, U4 STM32F373VBTx, U5 LM2904, U6 TCAN332, Y1 HSE, Y2 LSE

Commit message: Update CAN-bus configuration
Other:
- net class Default removed
